File: Gsm-Module-Kicad-Files/MICROCONTROLLER.sch (KiCad schematic (older format))
At the start: 22 parts, among them J2 Conn_01x05_Male, J3 USB_OTG, SW1 SW_Push, Y1 4-24 Mhz, Y2 32.768kHz

Commit message: edited
Parts:
- C9: symbol gsm-module-rescue:CP1-Device-gsm-module-rescue-gsm-module-rescue-gsm-module-rescue-gsm-module-rescue -> gsm-module-rescue:CP1-Device-gsm-module-rescue-gsm-module-rescue-gsm-module-rescue-gsm-module-rescue-gsm-module-rescue
- LQFP481: symbol gsm-module-rescue:NUC126LG4AE-NUC126LG4AE-gsm-module-rescue-gsm-module-rescue-gsm-module-rescue-gsm-module-rescue -> gsm-module-rescue:NUC126LG4AE-NUC126LG4AE-gsm-module-rescue-gsm-module-rescue-gsm-module-rescue-gsm-module-rescue-gsm-m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
Changed lines of the file:
@@
 	4650 2650 4850 2650
 $Comp
-L gsm-module-rescue:NUC126LG4AE-NUC126LG4AE-gsm-module-rescue-gsm-module-rescue-gsm-module-rescue-gsm-module-rescue LQFP481
+L gsm-module-rescue:NUC126LG4AE-NUC126LG4AE-gsm-module-rescue-gsm-module-rescue-gsm-module-rescue-gsm-module-rescue-gsm-module-rescue LQFP481
 U 1 1 6102037D
 P 8200 9100
@@
 Connection ~ 4450 4400
 $Comp
-L gsm-module-rescue:CP1-Device-gsm-module-rescue-gsm-module-rescue-gsm-module-rescue-gsm-module-rescue C9
+L gsm-module-rescue:CP1-Device-gsm-module-rescue-gsm-module-rescue-gsm-module-rescue-gsm-module-rescue-gsm-module-rescue C9
 U 1 1 61133DF4
 P 3500 4950
